Commit message: Twist to pwm and joystick

File: motor_controller/motor_controller/urdf/motor.urdf.xacro (robot description, xacro)
@@ -68,4 +68,19 @@
         </visual>
     </link>
+    <link name="rotor3">
+        <collision>
+            <origin xyz="0 0 -0.05" rpy="0 0 0" />
+            <geometry>
+                <cylinder radius="0.3" length="0.5" />
+            </geometry>
+        </collision>
+        <visual>
+            <origin xyz="0 0 0" rpy="0 0 0" />
+            <geometry>
+                <cylinder radius="0.3" length="0.5" />
+            </geometry>
+            <material name="red" />
+        </visual>
+    </link>
     <!-- Define joint named "joint1" with type "fixed" -->
     <joint name="joint1" type="fixed">
@@ -89,4 +104,10 @@
         <axis xyz="0 0 1" />
     </joint>
+    <joint name="joint4" type="continuous">
+        <parent link="base" />
+        <child link="rotor3" />
+        <origin xyz="-0.65 0 0.25" rpy="-0.5236 0 0" />
+        <axis xyz="0 0 1" />
+    </joint>
   <ros2_control name="arduino_actuator_ros2_control" type="system">
     <hardware>
@@ -106,4 +127,10 @@
         <state_interface name="position"/>
     </joint>
+    <joint name="joint4">
+        <command_interface name="velocity">
+        </command_interface>
+        <state_interface name="velocity"/>
+        <state_interface name="position"/>
+    </joint>
   </ros2_control>
 </robot>
